Commit message: rosbee_description -Adjusted Kinect Orientation -Tested with open_ni

File: trunk/ROS/rosbee_description/urdf/sensors/kinect/kinect.urdf.xacro (robot description, xacro)
@@ -26,5 +26,5 @@
     </link>
     <joint name="camera_rgb_optical_joint" type="fixed">
-      <origin xyz="0 0 0" rpy="${-M_PI/2} 0 ${-M_PI/2}" />
+      <origin xyz="0 0 0" rpy="${-M_PI/2} 0 0" />
       <parent link="camera_rgb_frame" />
       <child link="camera_rgb_optical_frame" />
@@ -40,5 +40,5 @@
     </link>
     <joint name="camera_joint" type="fixed">
-      <origin xyz="0 0 0" rpy="0 0 ${-M_PI/2}"/>
+      <origin xyz="0 0 0" rpy="0 0 0"/>
       <parent link="camera_rgb_frame"/>
       <child link="camera_link"/>
@@ -46,5 +46,5 @@
     <link name="camera_link">
       <visual>
-        <origin xyz="0 0 0" rpy="0 0 0"/>
+        <origin xyz="0 0 0" rpy="0 0 ${M_PI/2}"/>
         <geometry>
           <!--<box size="${kinect_length} ${kinect_width} ${kinect_height}"/>-->
