Commit message: rosbee_description - Added launch and urdf files for a simple representation of the rosbee robot - Simple model has been validated by measurements - Model with meshes still needs validation and adjustments

File: trunk/ROS/rosbee_description/robots/rosbee2a_simple.urdf.xacro (robot description, xacro)
@@ -10,7 +10,7 @@
   <include filename="$(find rosbee_description)/urdf/body/r2a_body.urdf.xacro" />
   <!-- Rosbee 2a pan tilt -->
-  <include filename="$(find rosbee_description)/urdf/misc/pan_tilt/pan_tilt.urdf.xacro" />
+  <include filename="$(find rosbee_description)/urdf/misc/pan_tilt/pan_tilt_simple.urdf.xacro" />
   <!-- Rosbee 2a kinect -->
-  <include filename="$(find rosbee_description)/urdf/sensors/kinect/kinect.urdf.xacro" />
+  <include filename="$(find rosbee_description)/urdf/sensors/kinect/kinect_simple.urdf.xacro" />
   <xacro:rosbee_base name="base"/>
   <xacro:r2a_body name="body" parent="base">
@@ -18,9 +18,8 @@
   </xacro:r2a_body>
   <xacro:pan_tilt_kinect name="pan_tilt" parent="body">
-    <origin xyz="0.1675 0 0.073" rpy="0 0 0"/>
+    <origin xyz="0.171 0.055 0.0715" rpy="0 0 0"/>
   </xacro:pan_tilt_kinect>
   <xacro:sensor_kinect parent="pan_tilt_yaw_link">
-    <origin xyz="-0.0011 -0.0003 0.03" rpy="0 0 0"/>
-    <!-- <origin xyz="-0.0011 -0.0003 0.03" rpy="0 0 0"/> -->
+    <origin xyz="0 0 0.0287" rpy="0 0 0"/> <!-- z = 38/2 + 8/2 + 5.7 -->
   </xacro:sensor_kinect>
 </robot>

File: trunk/ROS/rosbee_description/urdf/base/base.urdf.xacro (robot description, xacro)
@@ -7,9 +7,9 @@
   <!-- properties values for rosbee2a base -->
   <!-- base properties -->
-  <property name="base_length" value="0.010" />
+  <property name="base_length" value="0.009" />
   <property name="base_radius" value="0.240" />
-  <property name="base_height" value="0.101" />
+  <property name="base_height" value="0.101" /><!--distance floor to base plate + base_length/2-->
   <!-- side wheel properties -->
-  <property name="side_wheel_offset_y" value="0.2025" />
+  <property name="side_wheel_offset_y" value="0.202" />
   <property name="side_wheel_radius" value="0.0615" />
   <property name="side_wheel_length" value="0.020" />
@@ -43,7 +43,8 @@
       <visual>
         <geometry>
-          <cylinder length="${base_length}" radius="${base_radius}"/>
+          <!--<cylinder length="${base_length}" radius="${base_radius}"/>-->
+          <mesh filename="package://rosbee_description/meshes/rosbee_base.stl" scale="0.01 0.01 0.01"/>
         </geometry>
-        <origin rpy="0 0 0" xyz="0 0 0"/>
+        <origin rpy="${M_PI/2} 0 0" xyz="0 0 0"/>
         <material name="lightwood">
           <color rgba="0.8 0.729 0.568 1"/>

File: trunk/ROS/rosbee_description/urdf/body/r2a_body.urdf.xacro (robot description, xacro)
@@ -18,5 +18,4 @@
       <geometry>
         <box size="${body_length} ${body_width} ${body_height}"/>
-        <!--<mesh filename="package://pr2_description/meshes/torso_v0/torso_lift_L.stl"  />-->
       </geometry>
       <origin rpy="0 0 0" xyz="0 0 0"/>
