Commit message: Added Kinect to rosbee_description Kinect is still represented by a simple box

File: trunk/ROS/rosbee_description/robots/rosbee2a.urdf.xacro (robot description, xacro)
@@ -11,4 +11,6 @@
   <!-- Rosbee 2a pan tilt -->
   <include filename="$(find rosbee_description)/urdf/misc/pan_tilt/pan_tilt.urdf.xacro" />
+  <!-- Rosbee 2a kinect -->
+  <include filename="$(find rosbee_description)/urdf/sensors/kinect/kinect.urdf.xacro" />
   <xacro:rosbee_base name="base"/>
   <xacro:r2a_body name="body" parent="base">
@@ -18,3 +20,6 @@
     <origin xyz="0.1675 0.055 0.07" rpy="0 0 0"/>
   </xacro:pan_tilt_kinect>
+  <xacro:sensor_kinect parent="pan_tilt_yaw_link">
+    <origin xyz="0 0 0.03" rpy="0 0 0"/>
+  </xacro:sensor_kinect>
 </robot>

File: trunk/ROS/rosbee_description/urdf/misc/pan_tilt/pan_tilt.urdf.xacro (robot description, xacro)
@@ -37,12 +37,12 @@
     <link name="${name}_link">
       <visual>
-      <geometry>
-        <box size="${pan_tilt_length} ${pan_tilt_width} ${pan_tilt_height}"/>
-      </geometry>
-      <origin rpy="0 0 0" xyz="0 0 0"/>
-      <material name="darkblue">
-        <color rgba="0.0470 0.0039 0.5019 1"/>
-      </material>
-    </visual>
+        <geometry>
+          <box size="${pan_tilt_length} ${pan_tilt_width} ${pan_tilt_height}"/>
+        </geometry>
+        <origin rpy="0 0 0" xyz="0 0 0"/>
+        <material name="darkblue">
+          <color rgba="0.0470 0.0039 0.5019 1"/>
+        </material>
+      </visual>
     </link>
     <joint name="${name}_pitch_joint" type="revolute">
@@ -61,12 +61,12 @@
     <link name="${name}_pitch_link">
       <visual>
-      <geometry>
-        <box size="${pan_tilt_pitch_length} ${pan_tilt_pitch_width} ${pan_tilt_pitch_height}"/>
-      </geometry>
-      <origin rpy="0 0 0" xyz="0 0 0"/>
-      <material name="white">
-        <color rgba="1 1 1 1"/>
-      </material>
-    </visual>
+        <geometry>
+          <box size="${pan_tilt_pitch_length} ${pan_tilt_pitch_width} ${pan_tilt_pitch_height}"/>
+        </geometry>
+        <origin rpy="0 0 0" xyz="0 0 0"/>
+        <material name="white">
+          <color rgba="1 1 1 1"/>
+        </material>
+      </visual>
     </link>
     <joint name="${name}_yaw_joint" type="revolute">

Commit message: rosbee decription fixed body position

File: trunk/ROS/rosbee_description/robots/rosbee2a.urdf.xacro (robot description, xacro)
@@ -15,5 +15,5 @@
   <xacro:rosbee_base name="base"/>
   <xacro:r2a_body name="body" parent="base">
-    <origin xyz="0 0 0.045" rpy="0 0 0" />
+    <origin xyz="0 0 0.0495" rpy="0 0 0" />
   </xacro:r2a_body>
   <xacro:pan_tilt_kinect name="pan_tilt" parent="body">

Commit message: Added Meshes for pan-tilt and Kinect. Still experimental. URDF's might need restructuring.

File: trunk/ROS/rosbee_description/robots/rosbee2a.urdf.xacro (robot description, xacro)
@@ -18,8 +18,8 @@
   </xacro:r2a_body>
   <xacro:pan_tilt_kinect name="pan_tilt" parent="body">
-    <origin xyz="0.1675 0.055 0.07" rpy="0 0 0"/>
+    <origin xyz="0.1675 0 0.073" rpy="0 0 0"/>
   </xacro:pan_tilt_kinect>
   <xacro:sensor_kinect parent="pan_tilt_yaw_link">
-    <origin xyz="0 0 0.03" rpy="0 0 0"/>
+    <origin xyz="-0.0011 -0.0003 0.03" rpy="0 0 0"/>
   </xacro:sensor_kinect>
 </robot>

File: trunk/ROS/rosbee_description/urdf/misc/pan_tilt/pan_tilt.urdf.xacro (robot description, xacro)
@@ -14,6 +14,6 @@
   <property name="pan_tilt_pitch_height" value="0.043" />
   <property name="pan_tilt_pitch_offset_x" value="0.0" />
-  <property name="pan_tilt_pitch_offset_y" value="-0.064" />
-  <property name="pan_tilt_pitch_offset_z" value="0.017" />
+  <property name="pan_tilt_pitch_offset_y" value="-0.014" />
+  <property name="pan_tilt_pitch_offset_z" value="0.0157" />
   <property name="pan_tilt_pitch_velocity" value="0.5" />
   <property name="pan_tilt_pitch_lower" value="-${(M_PI/2)}" />
@@ -24,6 +24,6 @@
   <property name="pan_tilt_yaw_height" value="0.008" />
   <property name="pan_tilt_yaw_offset_x" value="0.0" />
-  <property name="pan_tilt_yaw_offset_y" value="0.005" />
-  <property name="pan_tilt_yaw_offset_z" value="0.0305" />
+  <property name="pan_tilt_yaw_offset_y" value="0.0125" />
+  <property name="pan_tilt_yaw_offset_z" value="0.017" />
   <property name="pan_tilt_yaw_velocity" value="0.5" />
   <property name="pan_tilt_yaw_lower" value="-${(M_PI)}" />
@@ -38,7 +38,8 @@
       <visual>
         <geometry>
-          <box size="${pan_tilt_length} ${pan_tilt_width} ${pan_tilt_height}"/>
+          <!--<box size="${pan_tilt_length} ${pan_tilt_width} ${pan_tilt_height}"/>-->
+          <mesh filename="package://rosbee_description/meshes/kinect_base_merged_pitch.stl" scale="0.001 0.001 0.001"/>
         </geometry>
-        <origin rpy="0 0 0" xyz="0 0 0"/>
+        <origin rpy="0 0 ${M_PI/2}" xyz="0 0 0"/>
         <material name="darkblue">
           <color rgba="0.0470 0.0039 0.5019 1"/>
@@ -62,7 +63,8 @@
       <visual>
         <geometry>
-          <box size="${pan_tilt_pitch_length} ${pan_tilt_pitch_width} ${pan_tilt_pitch_height}"/>
+          <!--<box size="${pan_tilt_pitch_length} ${pan_tilt_pitch_width} ${pan_tilt_pitch_height}"/>-->
+          <mesh filename="package://rosbee_description/meshes/kinect_base_merged_yaw.stl" scale="0.001 0.001 0.001"/>
         </geometry>
-        <origin rpy="0 0 0" xyz="0 0 0"/>
+        <origin rpy="0 0 ${M_PI/2}" xyz="0 0 0"/>
         <material name="white">
           <color rgba="1 1 1 1"/>
@@ -84,4 +86,5 @@
     </joint>
     <link name="${name}_yaw_link">
+      <!--
       <visual>
         <geometry>
@@ -93,4 +96,5 @@
         </material>
       </visual>
+      -->
     </link>
   </xacro:macro>

File: trunk/ROS/rosbee_description/urdf/sensors/kinect/kinect.urdf.xacro (robot description, xacro)
@@ -40,5 +40,5 @@
     </link>
     <joint name="camera_joint" type="fixed">
-      <origin xyz="0 0 0" rpy="0 0 0"/>
+      <origin xyz="0 0 0" rpy="0 0 ${-M_PI/2}"/>
       <parent link="camera_rgb_frame"/>
       <child link="camera_link"/>
@@ -48,8 +48,9 @@
         <origin xyz="0 0 0" rpy="0 0 0"/>
         <geometry>
-          <box size="${kinect_length} ${kinect_width} ${kinect_height}"/>
+          <!--<box size="${kinect_length} ${kinect_width} ${kinect_height}"/>-->
+          <mesh filename="package://rosbee_description/meshes/kinect_base_merged_kinect.stl" scale="0.001 0.001 0.001"/>
         </geometry>
-        <material name="black">
-          <color rgba="0 0 0 1"/>
+        <material name="white">
+          <color rgba="1 1 1 1"/>
         </material>
       </visual>

Commit message: rosbee_description -Added model with meshes

File: trunk/ROS/rosbee_description/robots/rosbee2a.urdf.xacro (robot description, xacro)
@@ -18,8 +18,8 @@
   </xacro:r2a_body>
   <xacro:pan_tilt_kinect name="pan_tilt" parent="body">
-    <origin xyz="0.1675 0 0.073" rpy="0 0 0"/>
+    <origin xyz="-0.1675 0 0.073" rpy="0 0 3.14"/>
   </xacro:pan_tilt_kinect>
   <xacro:sensor_kinect parent="pan_tilt_yaw_link">
-    <origin xyz="-0.0011 -0.0003 0.03" rpy="0 0 0"/>
+    <origin xyz="-0.0000 -0.0000 0.0287" rpy="0 0 3.14"/>
     <!-- <origin xyz="-0.0011 -0.0003 0.03" rpy="0 0 0"/> -->
   </xacro:sensor_kinect>

File: trunk/ROS/rosbee_description/urdf/misc/pan_tilt/pan_tilt.urdf.xacro (robot description, xacro)
@@ -14,6 +14,6 @@
   <property name="pan_tilt_pitch_height" value="0.043" />
   <property name="pan_tilt_pitch_offset_x" value="0.0" />
-  <property name="pan_tilt_pitch_offset_y" value="-0.014" />
-  <property name="pan_tilt_pitch_offset_z" value="0.0157" />
+  <property name="pan_tilt_pitch_offset_y" value="0.00" />
+  <property name="pan_tilt_pitch_offset_z" value="0.013" />
   <property name="pan_tilt_pitch_velocity" value="0.5" />
   <property name="pan_tilt_pitch_lower" value="-${(M_PI/2)}" />
@@ -23,7 +23,7 @@
   <property name="pan_tilt_yaw_length" value="0.040" />
   <property name="pan_tilt_yaw_height" value="0.008" />
-  <property name="pan_tilt_yaw_offset_x" value="0.0" />
-  <property name="pan_tilt_yaw_offset_y" value="0.0125" />
-  <property name="pan_tilt_yaw_offset_z" value="0.017" />
+  <property name="pan_tilt_yaw_offset_x" value="-0.0004" />
+  <property name="pan_tilt_yaw_offset_y" value="-0.0000" />
+  <property name="pan_tilt_yaw_offset_z" value="0.0300" />
   <property name="pan_tilt_yaw_velocity" value="0.5" />
   <property name="pan_tilt_yaw_lower" value="-${(M_PI)}" />
@@ -39,7 +39,7 @@
         <geometry>
           <!--<box size="${pan_tilt_length} ${pan_tilt_width} ${pan_tilt_height}"/>-->
-          <mesh filename="package://rosbee_description/meshes/kinect_base_merged_pitch.stl" scale="0.001 0.001 0.001"/>
+          <mesh filename="package://rosbee_description/meshes/pan_tilt_base.stl" scale="0.001 0.001 0.001"/>
         </geometry>
-        <origin rpy="0 0 ${M_PI/2}" xyz="0 0 0"/>
+        <origin rpy="0 0 ${M_PI}" xyz="0 0 0"/>
         <material name="darkblue">
           <color rgba="0.0470 0.0039 0.5019 1"/>
@@ -64,9 +64,9 @@
         <geometry>
           <!--<box size="${pan_tilt_pitch_length} ${pan_tilt_pitch_width} ${pan_tilt_pitch_height}"/>-->
-          <mesh filename="package://rosbee_description/meshes/kinect_base_merged_yaw.stl" scale="0.001 0.001 0.001"/>
+          <mesh filename="package://rosbee_description/meshes/pan_tilt_pitch.stl" scale="0.001 0.001 0.001"/>
         </geometry>
-        <origin rpy="0 0 ${M_PI/2}" xyz="0 0 0"/>
-        <material name="white">
-          <color rgba="1 1 1 1"/>
+        <origin rpy="0 0 ${M_PI}" xyz="0 0 0"/>
+        <material name="blue">
+          <color rgba="0.0470 0.0039 0.5019 1"/>
         </material>
       </visual>
@@ -86,15 +86,14 @@
     </joint>
     <link name="${name}_yaw_link">
-      <!--
       <visual>
         <geometry>
-          <box size="${pan_tilt_yaw_length} ${pan_tilt_yaw_width} ${pan_tilt_yaw_height}"/>
+          <!--<box size="${pan_tilt_yaw_length} ${pan_tilt_yaw_width} ${pan_tilt_yaw_height}"/>-->
+          <mesh filename="package://rosbee_description/meshes/pan_tilt_yaw.stl" scale="0.001 0.001 0.001"/>
         </geometry>
-        <origin rpy="0 0 0" xyz="0 0 0"/>
+        <origin rpy="0 0 ${M_PI}" xyz="0 0 0"/>
         <material name="white">
           <color rgba="1 1 1 1"/>
         </material>
       </visual>
-      -->
     </link>
   </xacro:macro>

File: trunk/ROS/rosbee_description/urdf/sensors/kinect/kinect.urdf.xacro (robot description, xacro)
@@ -46,11 +46,11 @@
     <link name="camera_link">
       <visual>
-        <origin xyz="0 0 0" rpy="0 0 ${M_PI/2}"/>
+        <origin xyz="0 0 0" rpy="0 0 0"/>
         <geometry>
           <!--<box size="${kinect_length} ${kinect_width} ${kinect_height}"/>-->
-          <mesh filename="package://rosbee_description/meshes/kinect_base_merged_kinect.stl" scale="0.001 0.001 0.001"/>
+          <mesh filename="package://rosbee_description/meshes/kinect.stl" scale="0.001 0.001 0.001"/>
         </geometry>
-        <material name="white">
-          <color rgba="1 1 1 1"/>
+        <material name="black">
+          <color rgba="0 0 0 1"/>
         </material>
       </visual>

Commit message: rosbee_description - fixed orientation

File: trunk/ROS/rosbee_description/robots/rosbee2a.urdf.xacro (robot description, xacro)
@@ -18,8 +18,8 @@
   </xacro:r2a_body>
   <xacro:pan_tilt_kinect name="pan_tilt" parent="body">
-    <origin xyz="-0.1675 0 0.073" rpy="0 0 3.14"/>
+    <origin xyz="-0.1675 0 0.073" rpy="0 0 0"/>
   </xacro:pan_tilt_kinect>
   <xacro:sensor_kinect parent="pan_tilt_yaw_link">
-    <origin xyz="-0.0000 -0.0000 0.0287" rpy="0 0 3.14"/>
+    <origin xyz="-0.0000 -0.0000 0.0287" rpy="0 0 0"/>
     <!-- <origin xyz="-0.0011 -0.0003 0.03" rpy="0 0 0"/> -->
   </xacro:sensor_kinect>

File: trunk/ROS/rosbee_description/urdf/misc/pan_tilt/pan_tilt.urdf.xacro (robot description, xacro)
@@ -25,5 +25,5 @@
   <property name="pan_tilt_yaw_offset_x" value="-0.0004" />
   <property name="pan_tilt_yaw_offset_y" value="-0.0000" />
-  <property name="pan_tilt_yaw_offset_z" value="0.0300" />
+  <property name="pan_tilt_yaw_offset_z" value="0.0295" />
   <property name="pan_tilt_yaw_velocity" value="0.5" />
   <property name="pan_tilt_yaw_lower" value="-${(M_PI)}" />
@@ -41,5 +41,5 @@
           <mesh filename="package://rosbee_description/meshes/pan_tilt_base.stl" scale="0.001 0.001 0.001"/>
         </geometry>
-        <origin rpy="0 0 ${M_PI}" xyz="0 0 0"/>
+        <origin rpy="0 0 0" xyz="0 0 0"/>
         <material name="darkblue">
           <color rgba="0.0470 0.0039 0.5019 1"/>
@@ -66,5 +66,5 @@
           <mesh filename="package://rosbee_description/meshes/pan_tilt_pitch.stl" scale="0.001 0.001 0.001"/>
         </geometry>
-        <origin rpy="0 0 ${M_PI}" xyz="0 0 0"/>
+        <origin rpy="0 0 0" xyz="0 0 0"/>
         <material name="blue">
           <color rgba="0.0470 0.0039 0.5019 1"/>
@@ -91,5 +91,5 @@
           <mesh filename="package://rosbee_description/meshes/pan_tilt_yaw.stl" scale="0.001 0.001 0.001"/>
         </geometry>
-        <origin rpy="0 0 ${M_PI}" xyz="0 0 0"/>
+        <origin rpy="0 0 0" xyz="0 0 0"/>
         <material name="white">
           <color rgba="1 1 1 1"/>

File: trunk/ROS/rosbee_description/urdf/sensors/kinect/kinect.urdf.xacro (robot description, xacro)
@@ -26,5 +26,5 @@
     </link>
     <joint name="camera_rgb_optical_joint" type="fixed">
-      <origin xyz="0 0 0" rpy="${-M_PI/2} 0 0" />
+      <origin xyz="0 0 0" rpy="${M_PI/2} 0 0" />
       <parent link="camera_rgb_frame" />
       <child link="camera_rgb_optical_frame" />
